Commit message: Actualización en modelos URDF y adiciónd de .gitignore

File: ros2_ws/src/s6_cpp_urdf/urdf/r2d2.urdf (robot description, URDF)
Before this commit: robot physics, 16 links, 15 joints
Links:
- added link base_footprint
- link left_gripper: geometry collision mesh filename=package://s6_cpp_urdf/meshes/l_finger.dae; visual mesh filename=package://s6_cpp_urdf/meshes/l_finger.dae
- link left_tip: geometry collision mesh filename=package://s6_cpp_urdf/meshes/l_finger_tip.dae; visual mesh filename=package://s6_cpp_urdf/meshes/l_finger_tip.dae
- link right_gripper: geometry collision mesh filename=package://s6_cpp_urdf/meshes/l_finger.dae; visual mesh filename=package://s6_cpp_urdf/meshes/l_finger.dae
- link right_tip: geometry collision mesh filename=package://s6_cpp_urdf/meshes/l_finger_tip.dae; visual mesh filename=package://s6_cpp_urdf/meshes/l_finger_tip.dae
Joints:
- added joint base_joint: type fixed, parent base_footprint, child base_link, origin xyz=0.0 0.0 0.47 rpy=0.0 0.0 0.0

File: ros2_ws/src/s6_cpp_urdf/urdf/r2d2_2.urdf (robot description, URDF)
Before this commit: robot r2d2, 7 links, 6 joints
Links:
- removed link axis
- added link base_footprint
- added link base_link; collision cylinder length=.5 radius=0.01; visual cylinder length=.5 radius=0.01
Joints:
- added joint base_joint: type fixed, parent base_footprint, child base_link, origin xyz=0.0 0.0 0.7 rpy=0.0 0.0 0.0
- joint leg1connect: parent axis -> base_link
- joint leg2connect: parent axis -> base_link
- joint tilt: parent axis -> base_link

File: ros2_ws/src/s6_py_urdf/urdf/r2d2.urdf (robot description, URDF)
Before this commit: robot physics, 16 links, 15 joints
Links:
- added link base_footprint
- link left_gripper: geometry collision mesh filename=package://s6_py_urdf/meshes/l_finger.dae; visual mesh filename=package://s6_py_urdf/meshes/l_finger.dae
- link left_tip: geometry collision mesh filename=package://s6_py_urdf/meshes/l_finger_tip.dae; visual mesh filename=package://s6_py_urdf/meshes/l_finger_tip.dae
- link right_gripper: geometry collision mesh filename=package://s6_py_urdf/meshes/l_finger.dae; visual mesh filename=package://s6_py_urdf/meshes/l_finger.dae
- link right_tip: geometry collision mesh filename=package://s6_py_urdf/meshes/l_finger_tip.dae; visual mesh filename=package://s6_py_urdf/meshes/l_finger_tip.dae
Joints:
- added joint base_joint: type fixed, parent base_footprint, child base_link, origin xyz=0.0 0.0 0.47 rpy=0.0 0.0 0.0
