Commit message: Correcting axis -> base_footprint link for R2D2 in s6_py_urdf and Updating path in URDF for .STL layers for s6_py_urdf

File: ros2_ws/src/s6_py_urdf/urdf/r2d2.urdf (robot description, URDF)
Before this commit: robot r2d2_physics, 17 links, 16 joints
Links:
- link left_gripper: geometry collision mesh filename=package://s6_py_urdf/meshes/l_finger.dae; visual mesh filename=package://s6_py_urdf/meshes/l_finger.dae
- link left_tip: geometry collision mesh filename=package://s6_py_urdf/meshes/l_finger_tip.dae; visual mesh filename=package://s6_py_urdf/meshes/l_finger_tip.dae
- link right_gripper: geometry collision mesh filename=package://s6_py_urdf/meshes/l_finger.dae; visual mesh filename=package://s6_py_urdf/meshes/l_finger.dae
- link right_tip: geometry collision mesh filename=package://s6_py_urdf/meshes/l_finger_tip.dae; visual mesh filename=package://s6_py_urdf/meshes/l_finger_tip.dae

File: ros2_ws/src/s6_py_urdf/urdf/rdk_x3_amr.urdf (robot description, URDF)
Before this commit: robot rdk_x3_robot, 10 links, 9 joints
Links:
- link base_link: geometry collision mesh filename=package://s6_py_urdf/meshes/base_link.STL; visual mesh filename=package://s6_py_urdf/meshes/base_link.STL
- link camera2_link: geometry collision mesh filename=package://s6_py_urdf/meshes/camera2_link.STL; visual mesh filename=package://s6_py_urdf/meshes/camera2_link.STL
- link camera_link: geometry collision mesh filename=package://s6_py_urdf/meshes/camera_link.STL; visual mesh filename=package://s6_py_urdf/meshes/camera_link.STL
- link imu_link: geometry collision mesh filename=package://s6_py_urdf/meshes/imu_link.STL; visual mesh filename=package://s6_py_urdf/meshes/imu_link.STL
- link left_back_wheel: geometry collision mesh filename=package://s6_py_urdf/meshes/left_back_wheel.STL; visual mesh filename=package://s6_py_urdf/meshes/left_back_wheel.STL
- link left_front_wheel: geometry collision mesh filename=package://s6_py_urdf/meshes/left_front_wheel.STL; visual mesh filename=package://s6_py_urdf/meshes/left_front_wheel.STL
- link lidar_link: geometry collision mesh filename=package://s6_py_urdf/meshes/lidar_link.STL; visual mesh filename=package://s6_py_urdf/meshes/lidar_link.STL
- link right_back_wheel: geometry collision mesh filename=package://s6_py_urdf/meshes/right_back_wheel.STL; visual mesh filename=package://s6_py_urdf/meshes/right_back_wheel.STL
- link right_front_wheel: geometry collision mesh filename=package://s6_py_urdf/meshes/right_front_wheel.STL; visual mesh filename=package://s6_py_urdf/meshes/right_front_wheel.STL
