Commit message: Refactoring cylinder robot model

File: ros2_ws/src/s8_py_slam/urdf/cylinder_plugin.urdf (robot description, URDF)
Before this commit: robot cylinder_robot, 7 links, 6 joints
Links:
- removed link front_marker
- added link base_link, mass 0.4728; collision box size=0.2 0.12 0.08; visual box size=0.2 0.12 0.08
- link left_back_wheel: mass 0.125 -> 0.05; geometry collision cylinder length=0.0306125 radius=0.0325; visual cylinder length=0.0306125 radius=0.0325
- link left_front_wheel: mass 0.125 -> 0.05; geometry collision cylinder length=0.0306125 radius=0.0325; visual cylinder length=0.0306125 radius=0.0325
- link lidar_link: mass 1.0 -> 0.0385; geometry collision cylinder length=0.033 radius=0.017; visual cylinder length=0.033 radius=0.017
- link right_back_wheel: mass 0.125 -> 0.05; geometry collision cylinder length=0.0306125 radius=0.0325; visual cylinder length=0.0306125 radius=0.0325
- link right_front_wheel: mass 0.125 -> 0.05; geometry collision cylinder length=0.0306125 radius=0.0325; visual cylinder length=0.0306125 radius=0.0325
Joints:
- removed joint front_marker_joint
- added joint base_joint: type fixed, parent base_footprint, child base_link, origin xyz=0 0 0.0625 rpy=0 0 0
- joint left_back_wheel_joint: origin xyz=-0.06 0.15 -0.06 rpy=0.0 0.0 0.0 -> xyz=-0.06 0.07655625 -0.03 rpy=0.0 0.0 0.0; parent lidar_link -> base_link
- joint left_front_wheel_joint: origin xyz=0.06 0.15 -0.06 rpy=0.0 0.0 0.0 -> xyz=0.06 0.07655625 -0.03 rpy=0.0 0.0 0.0; parent lidar_link -> base_link
- joint lidar_joint: origin xyz=0 0 0.11 rpy=0 0 0 -> xyz=0.06 0 0.0565 rpy=0 0 0; parent base_footprint -> base_link
- joint right_back_wheel_joint: origin xyz=-0.06 -0.15 -0.06 rpy=0.0 0.0 0.0 -> xyz=-0.06 -0.07655625 -0.03 rpy=0.0 0.0 0.0; parent lidar_link -> base_link
- joint right_front_wheel_joint: origin xyz=0.06 -0.15 -0.06 rpy=0.0 0.0 0.0 -> xyz=0.06 -0.07655625 -0.03 rpy=0.0 0.0 0.0; parent lidar_link -> base_link
