Commit message: Fixing AMR robot model for S8 pkg

File: ros2_ws/src/s8_py_slam/urdf/amr.urdf (robot description, URDF)
Before this commit: robot rdk_x3_amr, 10 links, 9 joints
Joints:
- joint base_joint: origin xyz=0.0 0.0 0.0659 rpy=0 0 0 -> xyz=0.0 0.0 0.06535 rpy=0 0 0
- joint left_back_joint: limit lower=0 upper=0 effort=0 velocity=0 -> (none)
- joint left_front_joint: limit lower=0 upper=0 effort=0 velocity=0 -> (none)
- joint right_back_joint: axis 0 -1 0 -> 0 1 0; limit lower=0 upper=0 effort=0 velocity=0 -> (none)
- joint right_front_joint: axis 0 -1 0 -> 0 1 0; limit lower=0 upper=0 effort=0 velocity=0 -> (none)

File: ros2_ws/src/s8_py_slam/urdf/amr_plugin.urdf (robot description, URDF)
Before this commit: robot rdk_x3_amr, 10 links, 9 joints
Joints:
- joint base_joint: origin xyz=0.0 0.0 0.0659 rpy=0 0 0 -> xyz=0.0 0.0 0.06535 rpy=0 0 0
- joint left_back_joint: limit lower=0 upper=0 effort=0 velocity=0 -> (none)
- joint left_front_joint: limit lower=0 upper=0 effort=0 velocity=0 -> (none)
- joint right_back_joint: axis 0 -1 0 -> 0 1 0; limit lower=0 upper=0 effort=0 velocity=0 -> (none)
- joint right_front_joint: axis 0 -1 0 -> 0 1 0; limit lower=0 upper=0 effort=0 velocity=0 -> (none)
